Commit message: update

File: vrx/vrx_2019/worlds/example_course.world.xacro (robot description, xacro)
@@ -9,24 +9,18 @@
     <xacro:ocean_waves/>
     <include>
-      <uri>model://robotx_navigation_challenge</uri>
-      <pose>58 68 2 0 0 0.4</pose>
+      <uri>model://obstacle_course0</uri>
+      <pose>66.66 122.88 0.157 0 0 -1.12</pose>
     </include>
     <include>
       <uri>model://robotx_light_buoy</uri>
-      <pose>110 28 0.25 0 0 0</pose>
+      <pose>113.6 84.68 0.37 0 0 0</pose>
     </include>
     <include>
-      <uri>model://robotx_2016_qualifying_pinger_transit</uri>
-      <pose>55 -50 0 0 0 -1.3</pose>
+      <uri>model://dock_2022</uri>
+      <pose>137.07 81.75 0.0 0 0 -1</pose>
     </include>
-    <!-- The 2016 dock with the three placards -->
     <include>
-      <uri>model://dock_2016</uri>
-      <pose>75 22 0.0 0 0 -2.78</pose>
-    </include>
-    <!-- The 2018 dock with the two placards -->
-    <include>
-      <uri>model://dock_2018</uri>
-      <pose>-2 -18 0.0 0 0 0.2</pose>
+      <uri>model://dock_2018_base_dynamic</uri>
+      <pose>114.44 73 -0.1585 -0.002089 0.000437 -1</pose>
     </include>
     <xacro:include filename="$(find vrx_gazebo)/worlds/xacros/usv_wind_plugin.xacro"/>
@@ -42,2 +36,14 @@
   </world>
 </sdf>
+    <!--<include>
+      <uri>model://obstacles_phase2_0</uri>
+      <pose>127 84 0.145 0 0 0.55</pose>
+    </include>-->
+    <!--<include>
+      <uri>model://obstacles_phase2_1</uri>
+      <pose>146 59 0 0 0 2.16</pose>
+    </include>-->
+     <!--<include>
+      <uri>model://obstacles_phase2_2</uri>
+      <pose>182 40 0.13 0 0 0 0.55</pose>
+    </include>-->

File: vrx/vrx_gazebo/worlds/xacros/usv_wind_plugin.xacro (robot description, xacro)
@@ -6,5 +6,5 @@
                          mean_vel:=0
                          var_gain:=0
-                         var_time:=2
+                         var_time:=20
                          seed:=''
                          ros_update_rate:=10

File: vrx/wamv_gazebo/urdf/wamv_gazebo.urdf.xacro (robot description, xacro)
@@ -9,5 +9,5 @@
   <xacro:arg name="imu_enabled" default="false" />
   <xacro:arg name="lidar_enabled" default="false" />
-  <xacro:arg name="ground_truth_enabled" default="false" />
+  <xacro:arg name="ground_truth_enabled" default="true" />
   <xacro:arg name="vrx_sensors_enabled" default="false" />
   <xacro:arg name="pinger_enabled" default="false" />
@@ -144,4 +144,5 @@
       <!-- Add pinger -->
       <xacro:wamv_pinger name="pinger" position="1.0 0 -1.0" />
+      <xacro:wamv_p3d name="p3d_wamv" />
       <!-- Add ball shooter (default pitch angle: ~-60 deg) -->
       <xacro:wamv_ball_shooter name="ball_shooter" x="0.54" y="0.30" z="1.296" pitch="-1.04"/>

File: vrx/wave_gazebo/world_models/ocean_waves/model.xacro (robot description, xacro)
@@ -17,5 +17,5 @@
 -->
 <world xmlns:xacro="http://ros.org/wiki/xacro">
-  <xacro:macro name="ocean_waves" params="gain:=0.1 period:=5
+  <xacro:macro name="ocean_waves" params="gain:=0.1 period:=0.1
                      direction_x:=1.0 direction_y:=0.0
                      angle:=0.4 scale:=1.5">
@@ -44,5 +44,5 @@
         <plugin name="ocean_waves_visual_plugin" filename="libWavefieldVisualPlugin.so">
           <enableRtt>true</enableRtt>
-          <rttNoise>0.1</rttNoise>
+          <rttNoise>0.1</rttNoise> <!-- for Camera -->
           <refractOpacity>0.2</refractOpacity>
           <reflectOpacity>0.2</reflectOpacity>
