Commit message: update-2

File: vrx/vrx_gazebo/worlds/xacros/usv_wind_plugin.xacro (robot description, xacro)
@@ -4,7 +4,7 @@
                params="**wind_objs
                          direction:=270
-                         mean_vel:=0
+                         mean_vel:=0.1
                          var_gain:=0
-                         var_time:=20
+                         var_time:=1000
                          seed:=''
                          ros_update_rate:=10

File: vrx/wamv_gazebo/urdf/wamv_gazebo.urdf.xacro (robot description, xacro)
@@ -9,5 +9,5 @@
   <xacro:arg name="imu_enabled" default="false" />
   <xacro:arg name="lidar_enabled" default="false" />
-  <xacro:arg name="ground_truth_enabled" default="true" />
+  <xacro:arg name="ground_truth_enabled" default="false" />
   <xacro:arg name="vrx_sensors_enabled" default="false" />
   <xacro:arg name="pinger_enabled" default="false" />
@@ -144,5 +144,4 @@
       <!-- Add pinger -->
       <xacro:wamv_pinger name="pinger" position="1.0 0 -1.0" />
-      <xacro:wamv_p3d name="p3d_wamv" />
       <!-- Add ball shooter (default pitch angle: ~-60 deg) -->
       <xacro:wamv_ball_shooter name="ball_shooter" x="0.54" y="0.30" z="1.296" pitch="-1.04"/>

File: vrx/wave_gazebo/world_models/ocean_waves/model.xacro (robot description, xacro)
@@ -17,5 +17,5 @@
 -->
 <world xmlns:xacro="http://ros.org/wiki/xacro">
-  <xacro:macro name="ocean_waves" params="gain:=0.1 period:=0.1
+  <xacro:macro name="ocean_waves" params="gain:=0.1 period:=0.01
                      direction_x:=1.0 direction_y:=0.0
                      angle:=0.4 scale:=1.5">
@@ -44,5 +44,5 @@
         <plugin name="ocean_waves_visual_plugin" filename="libWavefieldVisualPlugin.so">
           <enableRtt>true</enableRtt>
-          <rttNoise>0.1</rttNoise> <!-- for Camera -->
+          <rttNoise>0.1</rttNoise>
           <refractOpacity>0.2</refractOpacity>
           <reflectOpacity>0.2</reflectOpacity>
